File: STM32_mini/STM32_mini.kicad_pcb (KiCad board)
At the start: 2 copper layers, 52.5 x 51.5 mm, 33 parts, among them J1 Conn_01x04_Female, J2 Conn_01x05_Female, J3 Conn_01x04_Female, J4 USB_B_Micro, J5 Conn_01x02_Female, SW1 SW_Push, SW2 SW_SPDT, U1 STM32F030F4Px, U2 AMS1117-3.3, U3 CH340C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

Commit message: Overall Design Update
Parts:
- moved D3 4.07 mm to (162.1, 89.4), turned to 0 degrees
- moved R7 3.69 mm to (166.1, 89.4), turned to 180 degrees
- moved C10 0.60 mm to (136.3, 80.5)
- moved C5 0.50 mm to (157.7, 72.3)
- moved C1 0.40 mm to (146.4, 73.2)
- moved C2 0.40 mm to (144.6, 73.2)
- moved FB1 0.40 mm to (142.7, 73.5)
- moved C3 0.40 mm to (143.4, 78.5)
- moved C4 0.40 mm to (143.4, 76.7)
Connections:
- D3 pad 1: Net-(J2-Pad1) -> GND
- R7 pad 1: +3V3 -> Net-(J2-Pad1)
Routing:
- net GND: track 44.0 -> 47.8 mm, vias 12 -> 13
- net /NRST: track 35.1 -> 33.3 mm
- net Net-(J2-Pad1): track 29.8 -> 31.0 mm
- net +3V3: track 208.1 -> 209.1 mm
- net Net-(D3-Pad2): track 3.05 -> 2.24 mm
- net +3.3VA: track 6.67 -> 6.16 mm
- net (no net): vias 3 -> 4
