File: STM32_mini/STM32_mini.kicad_sch (KiCad schematic)
At the start: 37 parts, among them J1 Conn_01x04_Female, J2 Conn_01x05_Female, J3 Conn_01x04_Female, J4 USB_B_Micro, J5 Conn_01x02_Female, SW1 SW_Push, SW2 SW_SPDT, U1 STM32F030F4Px, U2 AMS1117-3.3, U3 CH340C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

Commit message: Overall Design Update
Connections:
- net +3V3: no longer R7.1
- net GND: now also D3.1 (K)
- net at J2.1 (Pin_1), U1.6 (PA0): now also R7.1; no longer D3.1 (K)
Other:
- moved on the sheet: D3, R7
Changed lines of the file:
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@@
-    (stroke (width 0) (type default) (color 0 0 0 0))
-  )
-  (wire (pts (xy 220.98 66.04) (xy 220.98 68.58))
     (stroke (width 0) (type default) (color 0 0 0 0))
   )
@@
     (stroke (width 0) (type default) (color 0 0 0 0))
   )
-  (wire (pts (xy 233.68 68.58) (xy 231.14 68.58))
+  (wire (pts (xy 231.14 66.04) (xy 233.68 66.04))
     (stroke (width 0) (type default) (color 0 0 0 0))
   )
@@
     (stroke (width 0) (type default) (color 0 0 0 0))
   )
-  (wire (pts (xy 243.84 68.58) (xy 241.3 68.58))
-    (stroke (width 0) (type default) (color 0 0 0 0))
-  )
   (wire (pts (xy 107.95 99.06) (xy 107.95 106.68))
     (stroke (width 0) (type default) (color 0 0 0 0))
@@
     (stroke (width 0) (type default) (color 0 0 0 0))
   )
-  (wire (pts (xy 220.98 68.58) (xy 223.52 68.58))
+  (wire (pts (xy 243.84 66.04) (xy 241.3 66.04))
     (stroke (width 0) (type default) (color 0 0 0 0))
   )
@@
     (stroke (width 0) (type default) (color 0 0 0 0))
   )
-  (wire (pts (xy 213.36 66.04) (xy 220.98 66.04))
+  (wire (pts (xy 213.36 66.04) (xy 223.52 66.04))
     (stroke (width 0) (type default) (color 0 0 0 0))
   )
@@
     (pin "1")
   )
-  (symbol (lib_id "Device:LED") (at 227.33 68.58 0) (unit 1)
+  (symbol (lib_id "Device:LED") (at 237.49 66.04 180) (unit 1)
     (in_bom yes) (on_board yes)
-    (property "Reference" "D3" (id 0) (at 224.79 66.802 0))
-    (property "Value" "LED" (id 1) (at 231.394 66.802 0))
-    (property "Footprint" "LED_SMD:LED_0805_2012Metric" (id 2) (at 227.33 68.58 0)
-      (effects (font (size 1.27 1.27)) hide)
-    )
-    (property "Datasheet" "~" (id 3) (at 227.33 68.58 0)
+    (property "Reference" "D3" (id 0) (at 240.03 67.818 0))
+    (property "Value" "LED" (id 1) (at 233.426 67.818 0))
+    (property "Footprint" "LED_SMD:LED_0805_2012Metric" (id 2) (at 237.49 66.04 0)
+      (effects (font (size 1.27 1.27)) hide)
+    )
+    (property "Datasheet" "~" (id 3) (at 237.49 66.04 0)
       (effects (font (size 1.27 1.27)) hide)
     )
@@
   (symbol (lib_id "Connector:Conn_01x05_Female") (at 218.44 73.66 0) (unit 1)
     (in_bom yes) (on_board yes)
-    (property "Reference" "J2" (id 0) (at 222.25 72.3899 0)
+    (property "Reference" "J2" (id 0) (at 217.424 81.28 0)
       (effects (font (size 1.27 1.27)) (justify left))
     )
@@
     (pin "2")
   )
-  (symbol (lib_id "power:+3V3") (at 243.84 68.58 0) (unit 1)
-    (in_bom yes) (on_board yes) (fields_autoplaced)
-    (property "Reference" "#PWR024" (id 0) (at 243.84 72.39 0)
-      (effects (font (size 1.27 1.27)) hide)
-    )
-    (property "Value" "+3V3" (id 1) (at 243.84 63.5 0))
-    (property "Footprint" "" (id 2) (at 243.84 68.58 0)
-      (effects (font (size 1.27 1.27)) hide)
-    )
-    (property "Datasheet" "" (id 3) (at 243.84 68.58 0)
-      (effects (font (size 1.27 1.27)) hide)
-    )
-    (pin "1")
-  )
   (symbol (lib_id "power:+3V3") (at 154.94 134.62 0) (unit 1)
     (in_bom yes) (on_board yes) (fields_autoplaced)
@@
     (pin "2")
   )
-  (symbol (lib_id "Device:R") (at 237.49 68.58 270) (unit 1)
+  (symbol (lib_id "Device:R") (at 227.33 66.04 90) (unit 1)
     (in_bom yes) (on_board yes)
-    (property "Reference" "R7" (id 0) (at 242.57 69.85 90))
-    (property "Value" "1k5" (id 1) (at 232.41 69.85 90))
-    (property "Footprint" "Resistor_SMD:R_0603_1608Metric" (id 2) (at 237.49 66.802 90)
-      (effects (font (size 1.27 1.27)) hide)
-    )
-    (property "Datasheet" "~" (id 3) (at 237.49 68.58 0)
+    (property "Reference" "R7" (id 0) (at 222.25 64.77 90))
+    (property "Value" "1k5" (id 1) (at 232.41 64.77 90))
+    (property "Footprint" "Resistor_SMD:R_0603_1608Metric" (id 2) (at 227.33 67.818 90)
+      (effects (font (size 1.27 1.27)) hide)
+    )
+    (property "Datasheet" "~" (id 3) (at 227.33 66.04 0)
       (effects (font (size 1.27 1.27)) hide)
     )
@@
     (pin "2")
   )
+  (symbol (lib_id "power:GND") (at 243.84 66.04 0) (mirror y) (unit 1)
+    (in_bom yes) (on_board yes) (fields_autoplaced)
+    (property "Reference" "#PWR0101" (id 0) (at 243.84 72.39 0)
+      (effects (font (size 1.27 1.27)) hide)
+    )
+    (property "Value" "GND" (id 1) (at 243.84 71.12 0)
+      (effects (font (size 1.27 1.27)) hide)
+    )
+    (property "Footprint" "" (id 2) (at 243.84 66.04 0)
+      (effects (font (size 1.27 1.27)) hide)
+    )
+    (property "Datasheet" "" (id 3) (at 243.84 66.04 0)
+      (effects (font (size 1.27 1.27)) hide)
+    )
+    (pin "1")
+  )
   (symbol (lib_id "Device:C") (at 129.54 54.61 0) (unit 1)
     (in_bom yes) (on_board yes) (fields_autoplaced)
@@
       (reference "#PWR023") (unit 1) (value "GND") (footprint "")
     )
-    (path "/c6eb2350-906d-4b0e-b96b-64a41dccae3a"
-      (reference "#PWR024") (unit 1) (value "+3V3") (footprint "")
-    )
     (path "/44311f9e-8be2-468f-aed9-04e963c8b05c"
       (reference "#PWR025") (unit 1) (value "+3V3") (footprint "")
@@
       (reference "#PWR026") (unit 1) (value "GND") (footprint "")
     )
+    (path "/f44b96e9-53da-488b-8ede-87d5b85d4c1e"
+      (reference "#PWR0101") (unit 1) (value "GND") (footprint "")
+    )
     (path "/ef357950-af6a-43cc-967e-f92d67b1d762"
